Commit message: bugfixes for apple_prediction node

File: harvest_hardware/realsense-ros/realsense2_description/urdf/_d435i.urdf.xacro (robot description, xacro)
@@ -22,6 +22,6 @@
   <xacro:include filename="$(find realsense2_description)/urdf/_d435.urdf.xacro"/>
   <xacro:include filename="$(find realsense2_description)/urdf/_d435i_imu_modules.urdf.xacro"/>
-  <xacro:macro name="sensor_d435i" params="parent *origin name:=camera use_nominal_extrinsics:=false">
-    <xacro:sensor_d435 parent="${parent}" name="${name}" use_nominal_extrinsics="${use_nominal_extrinsics}">
+  <xacro:macro name="sensor_d435i" params="parent *origin name:=camera use_nominal_extrinsics:=true">
+    <xacro:sensor_d435 parent="${parent}" name="${name}" use_nominal_extrinsics="true">
       <xacro:insert_block name="origin" />
     </xacro:sensor_d435>
