Commit message: added ur5e

File: harvest_hardware/ur5e_custom_hardware/urdf/gripper.urdf.xacro (robot description, xacro)
@@ -7,4 +7,17 @@
         <origin xyz="0.00 0 0.0" rpy="0 0 0"/>
     </joint>
+    <joint name="gripper_top_camera_joint" type="fixed">
+        <parent link="gripper_link"/>
+        <child link="gripper_top_camera_link"/>
+        <origin xyz="0.00 0 0.0" rpy="0 0 0"/>
+    </joint>
+    <link name="gripper_top_camera_link">
+        <visual>
+            <geometry>
+                <origin xyz="0.00 0 -0.085" rpy="0 0 0"/>
+                <box size="0.03 0.03 0.01"/>
+            </geometry>
+        </visual>
+    </link>
     <link name="gripper_palm_camera_link_optical">
         <visual>

Commit message: added realsense

File: harvest_hardware/ur5e_custom_hardware/urdf/gripper.urdf.xacro (robot description, xacro)
@@ -10,10 +10,9 @@
         <parent link="gripper_link"/>
         <child link="gripper_top_camera_link"/>
-        <origin xyz="0.00 0 0.0" rpy="0 0 0"/>
+        <origin xyz="0.00 -.08 -0.085" rpy="0 0 0"/>
     </joint>
     <link name="gripper_top_camera_link">
         <visual>
             <geometry>
-                <origin xyz="0.00 0 -0.085" rpy="0 0 0"/>
                 <box size="0.03 0.03 0.01"/>
             </geometry>
@@ -41,4 +40,9 @@
         </visual>
     </link>
+    <xacro:arg name="use_nominal_extrinsics" default="false" />
+    <xacro:include filename="$(find realsense2_description)/urdf/_d435i.urdf.xacro"/>
+    <xacro:sensor_d435i parent="gripper_top_camera_link" use_nominal_extrinsics="$(arg use_nominal_extrinsics)">
+      <origin xyz="0 0 0" rpy="0 -1.571 1.571"/>
+    </xacro:sensor_d435i>
 </xacro:macro>
 </robot>

Commit message: improved visual servoing code and added test node

File: harvest_hardware/ur5e_custom_hardware/urdf/gripper.urdf.xacro (robot description, xacro)
@@ -4,5 +4,5 @@
     <joint name="gripper_palm_camera_joint" type="fixed">
         <parent link="gripper_link"/>
-        <child link="gripper_palm_camera_link_optical"/>
+        <child link="gripper_palm_camera_optical_link"/>
         <origin xyz="0.00 0 0.0" rpy="0 0 0"/>
     </joint>
@@ -19,5 +19,5 @@
         </visual>
     </link>
-    <link name="gripper_palm_camera_link_optical">
+    <link name="gripper_palm_camera_optical_link">
         <visual>
             <geometry>

Commit message: added in harvest node, bugfixes, better launch files, more models, improved urdf

File: harvest_hardware/ur5e_custom_hardware/urdf/gripper.urdf.xacro (robot description, xacro)
@@ -5,17 +5,17 @@
         <parent link="gripper_link"/>
         <child link="gripper_palm_camera_optical_link"/>
-        <origin xyz="0.00 0 0.0" rpy="0 0 0"/>
+        <origin xyz="0.00 0 -0.05" rpy="0 0 0"/>
     </joint>
     <joint name="gripper_top_camera_joint" type="fixed">
         <parent link="gripper_link"/>
         <child link="gripper_top_camera_link"/>
-        <origin xyz="0.00 -.08 -0.085" rpy="0 0 0"/>
+        <origin xyz="0.00 -.072 -0.0865" rpy="0 0 0"/>
     </joint>
     <link name="gripper_top_camera_link">
-        <visual>
+        <!-- <collision>
             <geometry>
-                <box size="0.03 0.03 0.01"/>
+                <box size="0.08 0.05 0.01"/>
             </geometry>
-        </visual>
+        </collision> -->
     </link>
     <link name="gripper_palm_camera_optical_link">
@@ -24,4 +24,7 @@
                 <box size="0.03 0.03 0.01"/>
             </geometry>
+            <material name="green">
+                <color rgba="0 1 0 1"/>
+            </material>
         </visual>
     </link>
@@ -30,11 +33,11 @@
             <origin xyz="0.00 0 -0.105" rpy="0 0 0"/>
             <geometry>
-                <box size="0.06 0.06 0.2"/>
+                <box size="0.12 0.12 0.2"/>
             </geometry>
         </collision>
         <visual>
-            <origin xyz="0.00 0 -0.105" rpy="0 0 0"/>
+            <origin xyz="0.085 0 -0.2" rpy="0 0 3.14"/>
             <geometry>
-                <box size="0.06 0.06 0.2"/>
+                <mesh filename="package://ur5e_custom_hardware/meshes/03_mk3_full_assembly_coarse.STL" scale="0.001 0.001 0.001"/>
             </geometry>
         </visual>
