Commit message: final push before field trial 2025

File: harvest_hardware/robot_custom_hardware/urdf/cart_ur_gripper.urdf.xacro (robot description, xacro)
@@ -35,11 +35,9 @@
   <xacro:arg name="initial_positions_file" default="$(find robot_custom_hardware)/config/initial_positions.yaml"/>
   <xacro:property name="initial_positions_file" default="$(arg initial_positions_file)"/>
-  <!-- Amiga args -->
-  <xacro:arg name="amiga_prefix" default="amiga__"/>
-  <!-- Realsense args -->
+ <!-- Realsense args -->
   <xacro:arg name="use_nominal_extrinsics" default="true" />
   <!--Gripper Args-->
   <xacro:arg name="gripper_type" default="old"/>
-  <!-- Define the four args with the names the UR macro expects -->
+   <!-- Define the four args with the names the UR macro expects -->
   <xacro:arg name="joint_limit_params" default="$(find robot_custom_hardware)/config/ur5e/joint_limits.yaml"/>
   <xacro:arg name="kinematics_params"  default="$(find robot_custom_hardware)/config/ur5e/default_kinematics.yaml"/>
@@ -54,13 +52,27 @@
   <!-- define world exactly once -->
   <link name="world"/>
-  <!-- Instantiate Amiga, attached to world.
-       NOTE: your amiga macro signature requires mesh_base_path -->
-  <xacro:property name="robot_custom_hardware" value="package://robot_custom_hardware/"/>
-  <xacro:amiga_macro amiga_prefix="$(arg amiga_prefix)" amiga_parent="world" mesh_base_path="package://robot_custom_hardware/meshes/"/>
+  <!-- define cart -->
+  <link name="cart_body">
+    <collision>
+      <geometry>
+        <box size="0.8763 0.55404 0.86519" />
+      </geometry>
+    </collision>
+    <visual>
+      <geometry>
+        <box size="0.8763 0.55404 0.86519" />
+      </geometry>
+    </visual>
+  </link>
+  <joint name="body_joint" type="fixed" >
+    <parent link="world"/>
+    <child link="cart_body"/>
+    <origin xyz="0.00 0 0.43259" rpy="0 0 0" />
+  </joint>
   <!-- UR5e arm -->
   <xacro:ur_robot
       name="$(arg name)"
       tf_prefix="$(arg tf_prefix)"
-      parent="$(arg amiga_prefix)tool0"
+      parent="cart_body"
       joint_limits_parameters_file="$(arg joint_limit_params)"
       kinematics_parameters_file ="$(arg kinematics_params)"
@@ -95,5 +107,5 @@
       script_sender_port="$(arg script_sender_port)"
       trajectory_port="$(arg trajectory_port)">
-    <origin xyz="0 0 0" rpy="0 0 0"/>
+    <origin xyz="0 0 0.4326" rpy="0 0 0"/>
   </xacro:ur_robot>
   <!-- mount finray gripper -->
@@ -115,19 +127,6 @@
     <xacro:gripper_macro/> -->
   <!-- </xacro:if> -->
-  <!-- MAST Realsense for apple locations -->
-  <xacro:sensor_d435i
-    parent="$(arg amiga_prefix)base"
-    prefix="mast_"
-    use_nominal_extrinsics="$(arg use_nominal_extrinsics)">
-    <origin xyz="0.4064 -0.1778 1.5113" rpy="0 0 1.8852"/>
-  </xacro:sensor_d435i>
-  <!-- Realsense for trunk detections -->
-  <xacro:sensor_d435i
-    parent="$(arg amiga_prefix)base"
-    prefix="base_"
-    use_nominal_extrinsics="$(arg use_nominal_extrinsics)">
-    <origin xyz="0.0 0.3937 0.555625" rpy="0 0 1.57"/>
-  </xacro:sensor_d435i>
- <joint name="finray_tip" type="fixed">
+  <!-- Define link for manual apple location -->
+   <joint name="finray_tip" type="fixed">
       <parent link="tool0" />
       <child link="temp" />

File: harvest_hardware/robot_custom_hardware/urdf/finray_gripper.urdf.xacro (robot description, xacro)
@@ -21,5 +21,5 @@
             <parent link="finray_gripper_link" />
             <child link="gripper_palm_camera_optical_link" />
-            <origin xyz="0.00 0 0.024" rpy="0 0 0" />
+            <origin xyz="0.00 0 0.024" rpy="0 0 3.14159" />
         </joint>
         <!-- <joint name="finray_gripper_top_camera_joint" type="fixed">
@@ -53,5 +53,5 @@
                 <!-- <geometry>
                     <box size="0.12 0.12 0.2" />
-                </geometry> -->36
+                </geometry> -->
                 <!-- <geometry>
                     <cylinder length="0 .241" radius="0.110"/>
@@ -96,6 +96,8 @@
             prefix="gripper_"
             use_nominal_extrinsics="$(arg use_nominal_extrinsics)">
-            <origin xyz="-0.09 -0.06 -0.00875" rpy="0.5236 -1.5708 0"/>
-            <!-- <origin xyz="-0.065 -0.04075 -0.00875" rpy="0.5236 -1.5708 0"/> -->
+             <!-- move out for collision problem in intial collision body stl -->
+            <!-- <origin xyz="-0.09 -0.06 -0.00875" rpy="0.5236 -1.5708 0"/> -->
+            <!-- Aligned with model -->
+            <origin xyz="0.121651 -0.075874 -0.188703" rpy="2.618 -1.5708 0"/>
         </xacro:sensor_d435i>
         <!-- <xacro:arg name="use_nominal_extrinsics" default="false" />

Commit message: field Trial Changes

File: harvest_hardware/robot_custom_hardware/urdf/cart_ur_gripper.urdf.xacro (robot description, xacro)
@@ -124,6 +124,6 @@
       <child  link="gripper_link"/>
       <origin xyz="0.00 0.00 0.215" rpy="0 0 0"/>
-    </joint>
-    <xacro:gripper_macro/> -->
+    </joint> -->
+    <!-- <xacro:gripper_macro/> -->
   <!-- </xacro:if> -->
   <!-- Define link for manual apple location -->

File: harvest_hardware/robot_custom_hardware/urdf/gripper.urdf.xacro (robot description, xacro)
@@ -39,4 +39,13 @@
             </visual> -->
         </link>
+        <xacro:sensor_d435i
+            parent="gripper_link"
+            prefix="gripper_"
+            use_nominal_extrinsics="$(arg use_nominal_extrinsics)">
+             <!-- move out for collision problem in intial collision body stl -->
+            <!-- <origin xyz="-0.09 -0.06 -0.00875" rpy="0.5236 -1.5708 0"/> -->
+            <!-- Aligned with model -->
+            <origin xyz="0.121651 -0.075874 -0.188703" rpy="2.618 -1.5708 0"/>
+        </xacro:sensor_d435i>
         <link name="gripper_link">
             <collision>
