Commit message: cleans up launches for rviz and realsense, adds back in gripper_palm_camera script, launches move_arm again

File: harvest_hardware/harvest_hardware_description/urdf/amiga.urdf.xacro (robot description, xacro)
@@ -1,5 +1,5 @@
 <?xml version="1.0"?>
 <robot xmlns:xacro="https://ros.org/wiki/xacro" name="amiga">
-<xacro:macro name="amiga_macro" params="amiga_prefix:='amiga__' amiga_parent:='world' mesh_base_path">
+<xacro:macro name="amiga_macro" params="amiga_prefix:='amiga__' amiga_parent:='' mesh_base_path">
     <!-- ================== -->
     <!--     Amiga Macro    -->
@@ -107,9 +107,11 @@
     <!--       Joints       -->
     <!-- ================== -->
-    <joint name="${amiga_parent}--${amiga_prefix}base" type ="fixed">
+    <xacro:if value="${amiga_parent != ''}">
+    <joint name="${amiga_parent}--${amiga_prefix}base" type="fixed">
         <origin rpy="0 0 0" xyz="0 0 0"/>
         <parent link="${amiga_parent}"/>
         <child link="${amiga_prefix}base"/>
     </joint>
+    </xacro:if>
     <joint name="${amiga_prefix}base--${amiga_prefix}body" type="fixed">
         <origin rpy="0 0 0" xyz="0 0 0"/>

File: harvest_hardware/harvest_hardware_description/urdf/amiga_ur_gripper.urdf.xacro (robot description, xacro)
@@ -49,10 +49,8 @@
   <xacro:include filename="$(find harvest_hardware_description)/urdf/gripper.urdf.xacro"/>
   <xacro:include filename="$(find harvest_hardware_description)/urdf/_d435i.urdf.xacro"/>
-  <!-- define world exactly once -->
-  <link name="world"/>
   <!-- Instantiate Amiga, attached to world.
        NOTE: the amiga macro signature requires mesh_base_path -->
   <xacro:property name="harvest_hardware_description" value="package://harvest_hardware_description/"/>
-  <xacro:amiga_macro amiga_prefix="$(arg amiga_prefix)" amiga_parent="world" mesh_base_path="package://harvest_hardware_description/meshes/"/>
+  <xacro:amiga_macro amiga_prefix="$(arg amiga_prefix)" amiga_parent="" mesh_base_path="package://harvest_hardware_description/meshes/"/>
   <!-- UR5e arm -->
   <xacro:ur_robot
