Commit message: Prep for field trials

File: harvest_hardware/harvest_hardware_description/urdf/amiga.urdf.xacro (robot description, xacro)
@@ -19,5 +19,5 @@
     <xacro:property name="amiga_collision_box2_z" value='0.25' />
     <xacro:property name="amiga_tool0_mount_rotation" value="0.0 0.0 ${pi / 4}"/>
-    <xacro:property name="amiga_tool0_mount_position" value="-0.095 0.306 1.04775"/>
+    <xacro:property name="amiga_tool0_mount_position" value="0.0 0.306 1.041"/>
     <!-- ================== -->
     <!--       Links        -->

File: harvest_hardware/harvest_hardware_description/urdf/amiga_ur_gripper.urdf.xacro (robot description, xacro)
@@ -38,5 +38,6 @@
   <xacro:arg name="use_nominal_extrinsics" default="true" />
   <!--Gripper Args-->
-  <xacro:arg name="gripper_type" default="old"/>
+  <xacro:arg name="gripper_type" default="finray"/>
+  <xacro:property name="gripper_type" default="$(arg gripper_type)"/>
   <!-- parameter files -->
   <xacro:arg name="joint_limit_params" default="$(find ur_description)/config/$(arg ur_type)/joint_limits.yaml"/>
@@ -96,14 +97,21 @@
   </xacro:ur_robot>
   <!-- mount finray gripper -->
-  <!-- <xacro:if value="${'$(arg gripper_type)' == 'finray'}"> -->
-    <!-- <joint name="finray_gripper_joint" type="fixed">
+  <xacro:if value="${gripper_type == 'finray'}">
+    <joint name="finray_gripper_joint" type="fixed">
       <parent link="tool0"/>
-      <child  link="finray_gripper_link"/>
-      <origin xyz="0.00 0.00 0.23474" rpy="0 0 0"/>
+      <child  link="gripper_link"/>
+      <origin xyz="0.00 0.00 0.0" rpy="0 0 0"/>
     </joint>
-     <xacro:finray_gripper_macro/> -->
-  <!-- </xacro:if> -->
+    <xacro:finray_gripper_macro/>
+    <joint name="finray_tip" type="fixed">
+      <parent link="tool0" />
+      <child link="temp" />
+      <origin xyz="0.000 -0.00 0.32" rpy="0 0 -2.618" />
+    </joint>
+    <link name="temp">
+    </link>
+  </xacro:if>
   <!-- mount gripper -->
-  <!-- <xacro:if value="${'$(arg gripper_type)' == 'old'}"> -->
+  <xacro:if value="${gripper_type == 'alejo'}">
     <joint name="gripper_joint" type="fixed">
       <parent link="tool0"/>
@@ -112,5 +120,5 @@
     </joint>
     <xacro:gripper_macro/>
-  <!-- </xacro:if> -->
+  </xacro:if>
   <!-- MAST Realsense for apple locations -->
   <xacro:sensor_d435i
@@ -148,10 +156,3 @@
     </collision>
   </link>
- <!-- <joint name="finray_tip" type="fixed">
-      <parent link="tool0" />
-      <child link="temp" />
-      <origin xyz="0.000 -0.00 0.32" rpy="0 0 -2.618" />
-  </joint>
-  <link name="temp">
-  </link> -->
 </robot>

File: harvest_hardware/harvest_hardware_description/urdf/cart_ur_gripper.urdf.xacro (robot description, xacro)
@@ -121,5 +121,13 @@
       <origin xyz="0.00 0.00 0.0" rpy="0 0 0"/>
     </joint>
-     <xacro:finray_gripper_macro/>
+    <xacro:finray_gripper_macro/>
+    <!-- Define link for manual apple location -->
+    <joint name="finray_tip" type="fixed">
+        <parent link="tool0" />
+        <child link="temp" />
+        <origin xyz="0.000 -0.00 0.290" rpy="0 0 -2.618" />
+    </joint>
+    <link name="temp">
+    </link>
   </xacro:if>
   <!-- mount gripper -->
@@ -132,11 +140,3 @@
     <xacro:gripper_macro/>
   </xacro:if>
-  <!-- Define link for manual apple location -->
-   <joint name="finray_tip" type="fixed">
-      <parent link="tool0" />
-      <child link="temp" />
-      <origin xyz="0.000 -0.00 0.290" rpy="0 0 -2.618" />
-  </joint>
-  <link name="temp">
-  </link>
 </robot>
