Commit message: cleans robot state publisher and moveit launch patterns

File: harvest_hardware/harvest_hardware_description/urdf/amiga_ur_gripper.urdf.xacro (robot description, xacro)
@@ -111,5 +111,6 @@
     prefix="base_"
     use_nominal_extrinsics="$(arg use_nominal_extrinsics)">
-    <origin xyz="0.0 0.3937 0.555625" rpy="0 0 1.57"/>
+    <origin xyz="0.0 0.3937 0.555625" rpy="0 0 1.57"/> <!-- Realworld mount location -->
+    <!-- <origin xyz="0.7 -0.75 0.555625" rpy="0 0 -1.57"/> --> <!-- Location used for warthog placement (original 0.7 0.69 0.555625-->
   </xacro:sensor_d435i>
   <!-- Tracking marker frame -->
@@ -129,4 +130,7 @@
       </material>
     </visual>
+    <collision>
+      <geometry><box size="0.0 0.0 0.0"/></geometry>
+    </collision>
   </link>
 </robot>

Commit message: Correct package names, Minimal working/tested in sim.

File: harvest_hardware/harvest_hardware_description/urdf/amiga_ur_gripper.urdf.xacro (robot description, xacro)
@@ -49,5 +49,5 @@
   <xacro:include filename="$(find harvest_hardware_description)/urdf/amiga.urdf.xacro"/>
   <xacro:include filename="$(find ur_description)/urdf/ur_macro.xacro"/>
-  <xacro:include filename="$(find robot_custom_hardware)/urdf/finray_gripper.urdf.xacro"/>
+  <xacro:include filename="$(find harvest_hardware_description)/urdf/finray_gripper.urdf.xacro"/>
   <xacro:include filename="$(find harvest_hardware_description)/urdf/gripper.urdf.xacro"/>
   <xacro:include filename="$(find harvest_hardware_description)/urdf/_d435i.urdf.xacro"/>
@@ -97,19 +97,19 @@
   <!-- mount finray gripper -->
   <!-- <xacro:if value="${'$(arg gripper_type)' == 'finray'}"> -->
-    <joint name="finray_gripper_joint" type="fixed">
+    <!-- <joint name="finray_gripper_joint" type="fixed">
       <parent link="tool0"/>
       <child  link="finray_gripper_link"/>
       <origin xyz="0.00 0.00 0.23474" rpy="0 0 0"/>
     </joint>
-     <xacro:finray_gripper_macro/>
+     <xacro:finray_gripper_macro/> -->
   <!-- </xacro:if> -->
   <!-- mount gripper -->
   <!-- <xacro:if value="${'$(arg gripper_type)' == 'old'}"> -->
-    <!-- <joint name="gripper_joint" type="fixed">
+    <joint name="gripper_joint" type="fixed">
       <parent link="tool0"/>
       <child  link="gripper_link"/>
       <origin xyz="0.00 0.00 0.215" rpy="0 0 0"/>
     </joint>
-    <xacro:gripper_macro/> -->
+    <xacro:gripper_macro/>
   <!-- </xacro:if> -->
   <!-- MAST Realsense for apple locations -->
@@ -148,5 +148,5 @@
     </collision>
   </link>
- <joint name="finray_tip" type="fixed">
+ <!-- <joint name="finray_tip" type="fixed">
       <parent link="tool0" />
       <child link="temp" />
@@ -154,4 +154,4 @@
   </joint>
   <link name="temp">
-  </link>
+  </link> -->
 </robot>

File: harvest_hardware/harvest_hardware_description/urdf/cart_ur_gripper.urdf.xacro (robot description, xacro)
@@ -33,5 +33,5 @@
   <xacro:arg name="sim_ignition" default="false"/>
   <xacro:arg name="simulation_controllers" default=""/>
-  <xacro:arg name="initial_positions_file" default="$(find robot_custom_hardware)/config/initial_positions.yaml"/>
+  <xacro:arg name="initial_positions_file" default="$(find harvest_hardware_description)/config/initial_positions.yaml"/>
   <xacro:property name="initial_positions_file" default="$(arg initial_positions_file)"/>
  <!-- Realsense args -->
@@ -40,14 +40,14 @@
   <xacro:arg name="gripper_type" default="old"/>
    <!-- Define the four args with the names the UR macro expects -->
-  <xacro:arg name="joint_limit_params" default="$(find robot_custom_hardware)/config/ur5e/joint_limits.yaml"/>
-  <xacro:arg name="kinematics_params"  default="$(find robot_custom_hardware)/config/ur5e/default_kinematics.yaml"/>
-  <xacro:arg name="physical_params"    default="$(find robot_custom_hardware)/config/ur5e/physical_parameters.yaml"/>
-  <xacro:arg name="visual_params"      default="$(find robot_custom_hardware)/config/ur5e/visual_parameters.yaml"/>
+  <xacro:arg name="joint_limit_params" default="$(find harvest_hardware_description)/config/ur5e/joint_limits.yaml"/>
+  <xacro:arg name="kinematics_params"  default="$(find harvest_hardware_description)/config/ur5e/default_kinematics.yaml"/>
+  <xacro:arg name="physical_params"    default="$(find harvest_hardware_description)/config/ur5e/physical_parameters.yaml"/>
+  <xacro:arg name="visual_params"      default="$(find harvest_hardware_description)/config/ur5e/visual_parameters.yaml"/>
   <!-- includes -->
-  <xacro:include filename="$(find robot_custom_hardware)/urdf/amiga.urdf.xacro"/>
+  <xacro:include filename="$(find harvest_hardware_description)/urdf/amiga.urdf.xacro"/>
   <xacro:include filename="$(find ur_description)/urdf/ur_macro.xacro"/>
-  <xacro:include filename="$(find robot_custom_hardware)/urdf/finray_gripper.urdf.xacro"/>
-  <xacro:include filename="$(find robot_custom_hardware)/urdf/gripper.urdf.xacro"/>
-  <xacro:include filename="$(find robot_custom_hardware)/urdf/_d435i.urdf.xacro"/>
+  <xacro:include filename="$(find harvest_hardware_description)/urdf/finray_gripper.urdf.xacro"/>
+  <xacro:include filename="$(find harvest_hardware_description)/urdf/gripper.urdf.xacro"/>
+  <xacro:include filename="$(find harvest_hardware_description)/urdf/_d435i.urdf.xacro"/>
   <!-- define world exactly once -->
   <link name="world"/>

File: harvest_hardware/harvest_hardware_description/urdf/finray_gripper.urdf.xacro (robot description, xacro)
@@ -2,5 +2,5 @@
 <robot xmlns:xacro="http://www.ros.org/wiki/xacro">
     <xacro:macro name="finray_gripper_macro">
-    <xacro:include filename="$(find robot_custom_hardware)/urdf/_d435i.urdf.xacro"/>
+    <xacro:include filename="$(find harvest_hardware_description)/urdf/_d435i.urdf.xacro"/>
         <joint name="finray_gripper_scups_joint" type="fixed">
             <parent link="finray_gripper_link" />
@@ -59,5 +59,5 @@
                 <geometry>
                     <mesh
-                        filename="package://robot_custom_hardware/meshes/end_effectors/Fin_Ray-URDF_Collision_Body-Depth_Camera-Simplified.stl"
+                        filename="package://harvest_hardware_description/meshes/end_effectors/Fin_Ray-URDF_Collision_Body-Depth_Camera-Simplified.stl"
                         scale="0.0001 0.0001 0.0001" />
                 </geometry>
@@ -67,5 +67,5 @@
                 <geometry>
                     <mesh
-                        filename="package://robot_custom_hardware/meshes/end_effectors/Fin_Ray_2025-Gripper_Full_Assembly-Depth_Camera-Simplified.stl"
+                        filename="package://harvest_hardware_description/meshes/end_effectors/Fin_Ray_2025-Gripper_Full_Assembly-Depth_Camera-Simplified.stl"
                         scale="0.0001 0.0001 0.0001" />
                 </geometry>
