Commit message: new urdf

File: harvest_hardware/harvest_hardware_description/urdf/cart_ur_gripper.urdf.xacro (robot description, xacro)
@@ -118,5 +118,5 @@
       <parent link="tool0"/>
       <child  link="finray_gripper_link"/>
-      <origin xyz="0.00 0.00 0.23474" rpy="0 0 0"/>
+      <origin xyz="0.00 0.00 0.0" rpy="0 0 0"/>
     </joint>
      <xacro:finray_gripper_macro/>

File: harvest_hardware/harvest_hardware_description/urdf/finray_gripper.urdf.xacro (robot description, xacro)
@@ -6,5 +6,5 @@
             <parent link="finray_gripper_link" />
             <child link="gripper_scups_link" />
-            <origin xyz="0.000 -0.003 0.055" rpy="0 0 -2.618" />
+            <origin xyz="0.000 0.00 0.255" rpy="0 0 0.0" />
         </joint>
         <link name="gripper_scups_link">
@@ -21,5 +21,5 @@
             <parent link="finray_gripper_link" />
             <child link="gripper_palm_camera_optical_link" />
-            <origin xyz="0.00 0 0.024" rpy="0 0 3.14159" />
+            <origin xyz="0.00 0 0.230" rpy="0 0 1.5708" />
         </joint>
         <!-- <joint name="finray_gripper_top_camera_joint" type="fixed">
@@ -48,5 +48,5 @@
         <link name="finray_gripper_link">
             <collision>
-                <origin xyz="-0.01125 -0.012 -0.07725" rpy="1.5708 0  -0.5236" />
+                <origin xyz="0.0 0.0 0.001" rpy="0.0 0  3.14159" />
                 <!-- With out Depth camera  -->
                 <!-- <origin xyz="-0.0037 -0.0005 -0.0723" rpy="1.5708 0  -0.5236" />  -->
@@ -59,14 +59,14 @@
                 <geometry>
                     <mesh
-                        filename="package://harvest_hardware_description/meshes/end_effectors/Fin_Ray-URDF_Collision_Body-Depth_Camera-Simplified.stl"
-                        scale="0.0001 0.0001 0.0001" />
+                        filename="package://harvest_hardware_description/meshes/end_effectors/Finray2526-URDF-Collision.stl"
+                        scale="0.001 0.001 0.001" />
                 </geometry>
             </collision>
             <visual>
-                <origin xyz="0.0011  0.0017 -0.1846" rpy="1.5708 0 3.14" />
+                <origin xyz="0.0  0.0 0.030321" rpy="0.0 0 3.14159" />
                 <geometry>
                     <mesh
-                        filename="package://harvest_hardware_description/meshes/end_effectors/Fin_Ray_2025-Gripper_Full_Assembly-Depth_Camera-Simplified.stl"
-                        scale="0.0001 0.0001 0.0001" />
+                        filename="package://harvest_hardware_description/meshes/end_effectors/Finray2526-Assembly.stl"
+                        scale="0.001 0.001 0.001" />
                 </geometry>
                 <material name="ur5_blue">
@@ -99,5 +99,5 @@
             <!-- <origin xyz="-0.09 -0.06 -0.00875" rpy="0.5236 -1.5708 0"/> -->
             <!-- Aligned with model -->
-            <origin xyz="0.121651 -0.075874 -0.188703" rpy="2.618 -1.5708 0"/>
+            <origin xyz="0.070774 -0.122583 0.040471" rpy="2.094395 -1.5708 0"/>
         </xacro:sensor_d435i>
         <!-- <xacro:arg name="use_nominal_extrinsics" default="false" />

Commit message: Updated URDF with gripper type parameters

File: harvest_hardware/harvest_hardware_description/urdf/cart_ur_gripper.urdf.xacro (robot description, xacro)
@@ -38,5 +38,6 @@
   <xacro:arg name="use_nominal_extrinsics" default="true" />
   <!--Gripper Args-->
-  <xacro:arg name="gripper_type" default="old"/>
+  <xacro:arg name="gripper_type" default="finray"/>
+  <xacro:property name="gripper_type" default="$(arg gripper_type)"/>
    <!-- Define the four args with the names the UR macro expects -->
   <!-- <xacro:arg name="joint_limit_params" default="$(find harvest_hardware_description)/config/ur5e/joint_limits.yaml"/>
@@ -114,26 +115,26 @@
   </xacro:ur_robot>
   <!-- mount finray gripper -->
-  <!-- <xacro:if value="${'$(arg gripper_type)' == 'finray'}"> -->
+  <xacro:if value="${gripper_type == 'finray'}">
     <joint name="finray_gripper_joint" type="fixed">
       <parent link="tool0"/>
-      <child  link="finray_gripper_link"/>
+      <child  link="gripper_link"/>
       <origin xyz="0.00 0.00 0.0" rpy="0 0 0"/>
     </joint>
      <xacro:finray_gripper_macro/>
-  <!-- </xacro:if> -->
+  </xacro:if>
   <!-- mount gripper -->
-  <!-- <xacro:if value="${'$(arg gripper_type)' == 'old'}"> -->
-    <!-- <joint name="gripper_joint" type="fixed">
+  <xacro:if value="${gripper_type == 'alejo'}">
+    <joint name="gripper_joint" type="fixed">
       <parent link="tool0"/>
       <child  link="gripper_link"/>
       <origin xyz="0.00 0.00 0.215" rpy="0 0 0"/>
-    </joint> -->
-    <!-- <xacro:gripper_macro/> -->
-  <!-- </xacro:if> -->
+    </joint>
+    <xacro:gripper_macro/>
+  </xacro:if>
   <!-- Define link for manual apple location -->
    <joint name="finray_tip" type="fixed">
       <parent link="tool0" />
       <child link="temp" />
-      <origin xyz="0.000 -0.00 0.32" rpy="0 0 -2.618" />
+      <origin xyz="0.000 -0.00 0.290" rpy="0 0 -2.618" />
   </joint>
   <link name="temp">

File: harvest_hardware/harvest_hardware_description/urdf/finray_gripper.urdf.xacro (robot description, xacro)
@@ -4,5 +4,5 @@
     <xacro:include filename="$(find harvest_hardware_description)/urdf/_d435i.urdf.xacro"/>
         <joint name="finray_gripper_scups_joint" type="fixed">
-            <parent link="finray_gripper_link" />
+            <parent link="gripper_link" />
             <child link="gripper_scups_link" />
             <origin xyz="0.000 0.00 0.255" rpy="0 0 0.0" />
@@ -19,10 +19,10 @@
         </link>
         <joint name="finray_gripper_palm_camera_joint" type="fixed">
-            <parent link="finray_gripper_link" />
+            <parent link="gripper_link" />
             <child link="gripper_palm_camera_optical_link" />
             <origin xyz="0.00 0 0.230" rpy="0 0 1.5708" />
         </joint>
         <!-- <joint name="finray_gripper_top_camera_joint" type="fixed">
-            <parent link="finray_gripper_link" />
+            <parent link="gripper_link" />
             <child link="finray_gripper_top_camera_link" />
             <origin xyz="0.00 -.072 -0.0865" rpy="0 0 0" /> -->
@@ -46,5 +46,5 @@
             </visual>
         </link>
-        <link name="finray_gripper_link">
+        <link name="gripper_link">
             <collision>
                 <origin xyz="0.0 0.0 0.001" rpy="0.0 0  3.14159" />
@@ -93,5 +93,5 @@
         </link>
         <xacro:sensor_d435i
-            parent="finray_gripper_link"
+            parent="gripper_link"
             prefix="gripper_"
             use_nominal_extrinsics="$(arg use_nominal_extrinsics)">

File: harvest_hardware/harvest_hardware_moveit_config/srdf/ur.srdf.xacro (robot description, xacro)
@@ -5,5 +5,5 @@
   <!-- parameters -->
   <xacro:arg name="prefix" default="" />
-  <xacro:include filename="$(find ur_moveit_config)/srdf/ur_macro.srdf.xacro"/>
+  <xacro:include filename="$(find harvest_hardware_moveit_config)/srdf/ur_macro.srdf.xacro"/>
   <xacro:ur_srdf name="$(arg name)" prefix="$(arg prefix)"/>
 </robot>

File: harvest_hardware/harvest_hardware_moveit_config/srdf/ur_macro.srdf.xacro (robot description, xacro)
@@ -53,4 +53,6 @@
     <disable_collisions link1="${prefix}wrist_1_link" link2="${prefix}wrist_3_link" reason="Never" />
     <disable_collisions link1="${prefix}wrist_2_link" link2="${prefix}wrist_3_link" reason="Adjacent" />
+    <disable_collisions link1="${prefix}wrist_3_link" link2="gripper_link" reason="Adjacent" />
+    <disable_collisions link1="gripper_link" link2="gripper_camera_link" reason="Adjacent" />
   </xacro:macro>
 </robot>
