Commit message: Showing point cloud in launch file

File: harvest_hardware/harvest_hardware_description/urdf/_usb_palm.urdf.xacro (robot description, xacro)
@@ -1,32 +1,16 @@
 <?xml version="1.0"?>
 <!--
-# Copyright 2023 Intel Corporation. All Rights Reserved.
-#
-# Licensed under the Apache License, Version 2.0 (the "License");
-# you may not use this file except in compliance with the License.
-# You may obtain a copy of the License at
-#
-#     http://www.apache.org/licenses/LICENSE-2.0
-#
-# Unless required by applicable law or agreed to in writing, software
-# distributed under the License is distributed on an "AS IS" BASIS,
-# WITHOUT WARRANTIES OR CONDITIONS OF ANY KIND, either express or implied.
-# See the License for the specific language governing permissions and
-# limitations under the License.
+This is the URDF model for the palm camera, currently an ELP High Speed USB Camera, 1080P.
+1920 × 1080 (1080P): Up to 30 fps to 60 fps (MJPEG)
 -->
-<!--
-This is the URDF model for the Intel RealSense 435i camera, in it's
-aluminum peripherial evaluation case.
--->
-<robot name="sensor_d435i" xmlns:xacro="http://ros.org/wiki/xacro">
+<robot name="sensor_usb_palm" xmlns:xacro="http://ros.org/wiki/xacro">
   <xacro:include filename="$(find realsense2_description)/urdf/_d435.urdf.xacro"/>
   <xacro:include filename="$(find realsense2_description)/urdf/_d435i_imu_modules.urdf.xacro"/>
   <!-- Added prefix param -->
-  <xacro:macro name="sensor_d435i" params="parent prefix:='' *origin name:=camera use_nominal_extrinsics:=true">
+  <xacro:macro name="sensor_usb_palm" params="parent prefix:='' *origin name:=camera use_nominal_extrinsics:=true">
     <!-- Pass prefix to submodules -->
-    <xacro:sensor_d435 parent="${parent}" name="${prefix}${name}" use_nominal_extrinsics="${use_nominal_extrinsics}">
+    <xacro:sensor_usb_palm parent="${parent}" name="${prefix}${name}" use_nominal_extrinsics="${use_nominal_extrinsics}">
       <xacro:insert_block name="origin" />
-    </xacro:sensor_d435>
-    <xacro:d435i_imu_modules name="${prefix}${name}" use_nominal_extrinsics="${use_nominal_extrinsics}"/>
+    </xacro:sensor_usb_palm>
   </xacro:macro>
 </robot>
