Commit message: updated camera frames and harvest params

File: harvest_hardware/harvest_hardware_description/urdf/finray_gripper.urdf.xacro (robot description, xacro)
@@ -21,5 +21,5 @@
             <parent link="gripper_link" />
             <child link="gripper_palm_camera_optical_link" />
-            <origin xyz="0.00 0 0.230" rpy="0 0 1.5708" />
+            <origin xyz="0.00 0 0.230" rpy="0.0 0.0 -1.5708" />
         </joint>
         <!-- <joint name="finray_gripper_top_camera_joint" type="fixed">
