Commit message: Added action calls, and urdf parameters, need to test cancelability

File: harvest_hardware/harvest_hardware_moveit_config/srdf/ur.srdf.xacro (robot description, xacro)
@@ -5,4 +5,5 @@
   <!-- parameters -->
   <xacro:arg name="prefix" default="" />
+  <xacro:arg name="camera_mount" default="wrist"/>
   <xacro:include filename="$(find harvest_hardware_moveit_config)/srdf/ur_macro.srdf.xacro"/>
   <xacro:ur_srdf name="$(arg name)" prefix="$(arg prefix)"/>

File: harvest_hardware/harvest_hardware_moveit_config/srdf/ur_macro.srdf.xacro (robot description, xacro)
@@ -6,4 +6,6 @@
 -->
   <xacro:macro name="ur_srdf" params="name prefix">
+    <xacro:arg name="camera_mount" default="wrist"/>
+    <xacro:property name="camera_mount" default="$(arg camera_mount)"/>
     <!--GROUPS - Representation of a set of joints and links. This can be useful for specifying DOF to plan for, defining arms, end effectors, etc-->
     <!--LINKS - When a link is specified, the parent joint of that link (if it exists) is automatically included-->
@@ -54,5 +56,7 @@
     <disable_collisions link1="${prefix}wrist_2_link" link2="${prefix}wrist_3_link" reason="Adjacent" />
     <disable_collisions link1="${prefix}wrist_3_link" link2="gripper_link" reason="Adjacent" />
-    <disable_collisions link1="gripper_link" link2="gripper_camera_link" reason="Adjacent" />
+    <xacro:if value="${camera_mount == 'wrist'}">
+      <disable_collisions link1="gripper_link" link2="gripper_camera_link" reason="Adjacent" />
+    </xacro:if>
   </xacro:macro>
 </robot>
